File: IN_OUT.kicad_sch (KiCad schematic)
At the start: 33 parts, among them J4 8P8C_DS1134, J5 Conn_DEGSON_01x02_Pin, J6 Conn_DEGSON_01x02_Pin, J7 Conn_DEGSON_01x02_Pin, J8 Conn_DEGSON_01x02_Pin

Commit message: 32kHz replaced
Changed lines of the file:
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@@
 	(wire
 		(pts
-			(xy 118.11 180.34) (xy 121.92 180.34)
+			(xy 59.69 180.34) (xy 121.92 180.34)
 		)
 		(stroke
@@
 	(wire
 		(pts
-			(xy 74.93 43.18) (xy 81.28 43.18)
+			(xy 59.69 43.18) (xy 81.28 43.18)
 		)
 		(stroke
@@
 	(hierarchical_label "SENSOR_POWER"
 		(shape input)
-		(at 74.93 43.18 180)
+		(at 59.69 43.18 180)
 		(effects
 			(font
@@
 	(hierarchical_label "VBAT_LEVEL"
 		(shape output)
-		(at 118.11 180.34 180)
+		(at 59.69 180.34 180)
 		(effects
 			(font
@@
 		(dnp no)
 		(fields_autoplaced yes)
-		(property "Reference" "#PWR042"
+		(property "Reference" "#PWR043"
 			(at 121.92 198.12 0)
 			(effects
@@
 			(project "GSMtransmitter"
 				(path "/bbc92722-7b85-49e8-a662-589426df605a/72572aab-46c4-4091-abb3-71d2258d66fa"
-					(reference "#PWR042")
+					(reference "#PWR043")
 					(unit 1)
 				)
@@
 		(dnp no)
 		(fields_autoplaced yes)
-		(property "Reference" "#PWR041"
+		(property "Reference" "#PWR042"
 			(at 81.28 175.26 0)
 			(effects
@@
 			(project "GSMtransmitter"
 				(path "/bbc92722-7b85-49e8-a662-589426df605a/72572aab-46c4-4091-abb3-71d2258d66fa"
-					(reference "#PWR041")
+					(reference "#PWR042")
 					(unit 1)
 				)
@@
 		(dnp no)
 		(fields_autoplaced yes)
-		(property "Reference" "#PWR049"
+		(property "Reference" "#PWR050"
 			(at 181.61 132.08 0)
 			(effects
@@
 			(project "GSMtransmitter"
 				(path "/bbc92722-7b85-49e8-a662-589426df605a/72572aab-46c4-4091-abb3-71d2258d66fa"
-					(reference "#PWR049")
+					(reference "#PWR050")
 					(unit 1)
 				)
@@
 		(dnp no)
 		(fields_autoplaced yes)
-		(property "Reference" "#PWR053"
+		(property "Reference" "#PWR054"
 			(at 182.88 50.8 0)
 			(effects
@@
 			(project "GSMtransmitter"
 				(path "/bbc92722-7b85-49e8-a662-589426df605a/72572aab-46c4-4091-abb3-71d2258d66fa"
-					(reference "#PWR053")
+					(reference "#PWR054")
 					(unit 1)
 				)
@@
 		(dnp no)
 		(fields_autoplaced yes)
-		(property "Reference" "#PWR045"
+		(property "Reference" "#PWR046"
 			(at 149.86 71.12 0)
 			(effects
@@
 			(project "GSMtransmitter"
 				(path "/bbc92722-7b85-49e8-a662-589426df605a/72572aab-46c4-4091-abb3-71d2258d66fa"
-					(reference "#PWR045")
+					(reference "#PWR046")
 					(unit 1)
 				)
@@
 		(dnp no)
 		(fields_autoplaced yes)
-		(property "Reference" "#PWR052"
+		(property "Reference" "#PWR053"
 			(at 182.88 45.72 0)
 			(effects
@@
 			(project "GSMtransmitter"
 				(path "/bbc92722-7b85-49e8-a662-589426df605a/72572aab-46c4-4091-abb3-71d2258d66fa"
-					(reference "#PWR052")
+					(reference "#PWR053")
 					(unit 1)
 				)
@@
 		(dnp no)
 		(fields_autoplaced yes)
-		(property "Reference" "#PWR037"
+		(property "Reference" "#PWR038"
 			(at 81.28 100.33 0)
 			(effects
@@
 			(project "GSMtransmitter"
 				(path "/bbc92722-7b85-49e8-a662-589426df605a/72572aab-46c4-4091-abb3-71d2258d66fa"
-					(reference "#PWR037")
+					(reference "#PWR038")
 					(unit 1)
 				)
@@
 		(on_board yes)
 		(dnp no)
-		(property "Reference" "#PWR043"
+		(property "Reference" "#PWR044"
 			(at 135.89 172.72 0)
 			(effects
@@
 			(project "GSMtransmitter"
 				(path "/bbc92722-7b85-49e8-a662-589426df605a/72572aab-46c4-4091-abb3-71d2258d66fa"
-					(reference "#PWR043")
+					(reference "#PWR044")
 					(unit 1)
 				)
@@
 		(dnp no)
 		(fields_autoplaced yes)
-		(property "Reference" "#PWR050"
+		(property "Reference" "#PWR051"
 			(at 187.96 72.39 0)
 			(effects
@@
 			(project "GSMtransmitter"
 				(path "/bbc92722-7b85-49e8-a662-589426df605a/72572aab-46c4-4091-abb3-71d2258d66fa"
-					(reference "#PWR050")
+					(reference "#PWR051")
 					(unit 1)
 				)
@@
 		(dnp no)
 		(fields_autoplaced yes)
-		(property "Reference" "#PWR039"
+		(property "Reference" "#PWR040"
 			(at 81.28 137.16 0)
 			(effects
@@
 			(project "GSMtransmitter"
 				(path "/bbc92722-7b85-49e8-a662-589426df605a/72572aab-46c4-4091-abb3-71d2258d66fa"
-					(reference "#PWR039")
+					(reference "#PWR040")
 					(unit 1)
 				)
@@
 		(on_board yes)
 		(dnp no)
-		(property "Reference" "#PWR034"
+		(property "Reference" "#PWR035"
 			(at 81.28 35.56 0)
 			(effects
@@
 			(project "GSMtransmitter"
 				(path "/bbc92722-7b85-49e8-a662-589426df605a/72572aab-46c4-4091-abb3-71d2258d66fa"
-					(reference "#PWR034")
+					(reference "#PWR035")
 					(unit 1)
 				)
@@
 		(dnp no)
 		(fields_autoplaced yes)
-		(property "Reference" "#PWR031"
+		(property "Reference" "#PWR032"
 			(at 63.5 100.33 0)
 			(effects
@@
 			(project "GSMtransmitter"
 				(path "/bbc92722-7b85-49e8-a662-589426df605a/72572aab-46c4-4091-abb3-71d2258d66fa"
-					(reference "#PWR031")
+					(reference "#PWR032")
 					(unit 1)
 				)
@@
 		(dnp no)
 		(fields_autoplaced yes)
-		(property "Reference" "#PWR048"
+		(property "Reference" "#PWR049"
 			(at 170.18 111.76 0)
 			(effects
@@
 			(project "GSMtransmitter"
 				(path "/bbc92722-7b85-49e8-a662-589426df605a/72572aab-46c4-4091-abb3-71d2258d66fa"
-					(reference "#PWR048")
+					(reference "#PWR049")
 					(unit 1)
 				)
@@
 		(dnp no)
 		(fields_autoplaced yes)
-		(property "Reference" "#PWR044"
+		(property "Reference" "#PWR045"
 			(at 135.89 198.12 0)
 			(effects
@@
 			(project "GSMtransmitter"
 				(path "/bbc92722-7b85-49e8-a662-589426df605a/72572aab-46c4-4091-abb3-71d2258d66fa"
-					(reference "#PWR044")
+					(reference "#PWR045")
 					(unit 1)
 				)
@@
 		(dnp no)
 		(fields_autoplaced yes)
-		(property "Reference" "#PWR033"
+		(property "Reference" "#PWR034"
 			(at 63.5 175.26 0)
 			(effects
@@
 			(project "GSMtransmitter"
 				(path "/bbc92722-7b85-49e8-a662-589426df605a/72572aab-46c4-4091-abb3-71d2258d66fa"
-					(reference "#PWR033")
+					(reference "#PWR034")
 					(unit 1)
 				)
@@
 		(on_board yes)
 		(dnp no)
-		(property "Reference" "#PWR038"
+		(property "Reference" "#PWR039"
 			(at 81.28 111.76 0)
 			(effects
@@
 			(project "GSMtransmitter"
 				(path "/bbc92722-7b85-49e8-a662-589426df605a/72572aab-46c4-4091-abb3-71d2258d66fa"
-					(reference "#PWR038")
+					(reference "#PWR039")
 					(unit 1)
 				)
@@
 		(on_board yes)
 		(dnp no)
-		(property "Reference" "#PWR040"
+		(property "Reference" "#PWR041"
 			(at 81.28 149.86 0)
 			(effects
@@
 			(project "GSMtransmitter"
 				(path "/bbc92722-7b85-49e8-a662-589426df605a/72572aab-46c4-4091-abb3-71d2258d66fa"
-					(reference "#PWR040")
+					(reference "#PWR041")
 					(unit 1)
 				)
@@
 		(dnp no)
 		(fields_autoplaced yes)
-		(property "Reference" "#PWR047"
+		(property "Reference" "#PWR048"
 			(at 166.37 71.12 0)
 			(effects
@@
 			(project "GSMtransmitter"
 				(path "/bbc92722-7b85-49e8-a662-589426df605a/72572aab-46c4-4091-abb3-71d2258d66fa"
-					(reference "#PWR047")
+					(reference "#PWR048")
 					(unit 1)
 				)
@@
 		(dnp no)
 		(fields_autoplaced yes)
-		(property "Reference" "#PWR035"
+		(property "Reference" "#PWR036"
 			(at 81.28 60.96 0)
 			(effects
@@
 			(project "GSMtransmitter"
 				(path "/bbc92722-7b85-49e8-a662-589426df605a/72572aab-46c4-4091-abb3-71d2258d66fa"
-					(reference "#PWR035")
+					(reference "#PWR036")
 					(unit 1)
 				)
@@
 		(dnp no)
 		(fields_autoplaced yes)
-		(property "Reference" "#PWR032"
+		(property "Reference" "#PWR033"
 			(at 63.5 137.16 0)
 			(effects
@@
 			(project "GSMtransmitter"
 				(path "/bbc92722-7b85-49e8-a662-589426df605a/72572aab-46c4-4091-abb3-71d2258d66fa"
-					(reference "#PWR032")
+					(reference "#PWR033")
 					(unit 1)
 				)
@@
 		(dnp no)
 		(fields_autoplaced yes)
-		(property "Reference" "#PWR051"
+		(property "Reference" "#PWR052"
 			(at 182.88 40.64 0)
 			(effects
@@
 			(project "GSMtransmitter"
 				(path "/bbc92722-7b85-49e8-a662-589426df605a/72572aab-46c4-4091-abb3-71d2258d66fa"
-					(reference "#PWR051")
+					(reference "#PWR052")
 					(unit 1)
 				)
@@
 		(dnp no)
 		(fields_autoplaced yes)
-		(property "Reference" "#PWR046"
+		(property "Reference" "#PWR047"
 			(at 151.13 198.12 0)
 			(effects
@@
 			(project "GSMtransmitter"
 				(path "/bbc92722-7b85-49e8-a662-589426df605a/72572aab-46c4-4091-abb3-71d2258d66fa"
-					(reference "#PWR046")
+					(reference "#PWR047")
 					(unit 1)
 				)
@@
 		(on_board yes)
 		(dnp no)
-		(property "Reference" "#PWR036"
+		(property "Reference" "#PWR037"
 			(at 81.28 74.93 0)
 			(effects
@@
 			(project "GSMtransmitter"
 				(path "/bbc92722-7b85-49e8-a662-589426df605a/72572aab-46c4-4091-abb3-71d2258d66fa"
-					(reference "#PWR036")
+					(reference "#PWR037")
 					(unit 1)
 				)
