File: IN_OUT.kicad_sch (KiCad schematic)
At the start: 33 parts, among them J4 8P8C_DS1134, J5 Conn_DEGSON_01x02_Pin, J6 Conn_DEGSON_01x02_Pin, J7 Conn_DEGSON_01x02_Pin, J8 Conn_DEGSON_01x02_Pin

Commit message: Dual SIM version
Parts:
- removed C15: 100nF, Capacitor_SMD:C_0805_2012Metric_Pad1.18x1.45mm_HandSolder, symbol Device:C
- removed C16: 1000uFx35V, Capacitor_THT:CP_Radial_D12.5mm_P5.00mm, symbol Device:C_Polarized
- removed C17: 470nFx50V, Capacitor_SMD:C_0805_2012Metric_Pad1.18x1.45mm_HandSolder, symbol Device:C
- removed D15, D16: MBR0580, Diode_SMD:D_SOD-123, symbol Diode:MBR0580
- removed D17: SS26, Diode_SMD:D_SMA, symbol Diode:SS26
- removed J8: Conn_DEGSON_01x02_Pin, footprints:DEGSON_DG390-5.0-02P_1x02_P5.0mm_Vertical, symbol symbols:Conn_DEGSON_01x02_Pin
- removed R23: 100k, Resistor_SMD:R_0805_2012Metric_Pad1.20x1.40mm_HandSolder, symbol Device:R
- removed R24: 1M, Resistor_SMD:R_0805_2012Metric_Pad1.20x1.40mm_HandSolder, symbol Device:R
- C1: renamed from C12; MPN (none) -> CC0805KRX7R8BB104; Manufacturer (none) -> YAGEO
- C2: renamed from C13; MPN (none) -> CC0805KRX7R8BB104; Manufacturer (none) -> YAGEO
- C3: renamed from C14; MPN (none) -> CC0805KRX7R8BB104; Manufacturer (none) -> YAGEO
- D1: renamed from D7; MPN (none) -> MBR0580; Manufacturer (none) -> MCC
- D2: renamed from D8; MPN (none) -> MBR0580; Manufacturer (none) -> MCC
- D3: renamed from D9; MPN (none) -> MBR0580; Manufacturer (none) -> MCC
- D4: renamed from D10; MPN (none) -> MBR0580; Manufacturer (none) -> MCC
- D5: renamed from D11; MPN (none) -> MBR0580; Manufacturer (none) -> MCC
- D6: renamed from D12; MPN (none) -> MBR0580; Manufacturer (none) -> MCC
- D7: renamed from D13; MPN (none) -> MBR0580; Manufacturer (none) -> MCC
- D8: renamed from D14; MPN (none) -> MBR0580; Manufacturer (none) -> MCC
- J1: renamed from J4; value 8P8C_DS1134 -> DS1134-S80BPX; MPN (none) -> DS1134-S80BPX; Manufacturer (none) -> CONNFLY ELECTRONIC CO. LTD
- J2: renamed from J5; MPN (none) -> DG390-5.0-02P; Manufacturer (none) -> NINGBO DEGSON ELECTRICAL CO.,LTD.
- J3: renamed from J6; MPN (none) -> DG390-5.0-02P; Manufacturer (none) -> NINGBO DEGSON ELECTRICAL CO.,LTD.
- J4: renamed from J7; MPN (none) -> DG390-5.0-02P; Manufacturer (none) -> NINGBO DEGSON ELECTRICAL CO.,LTD.
- R1: renamed from R14; MPN (none) -> RC0805JR-07150KL; Manufacturer (none) -> YAGEO
- R2: renamed from R15; MPN (none) -> RC0805JR-07150KL; Manufacturer (none) -> YAGEO
- R3: renamed from R16; MPN (none) -> RC0805JR-07150KL; Manufacturer (none) -> YAGEO
- R4: renamed from R17; MPN (none) -> RC0805JR-074K7L; Manufacturer (none) -> YAGEO
- R5: renamed from R18; MPN (none) -> RC0805JR-074K7L; Manufacturer (none) -> YAGEO
- R6: renamed from R19; MPN (none) -> RC0805JR-074K7L; Manufacturer (none) -> YAGEO
- R7: renamed from R20; MPN (none) -> RC0805FR-0710KL; Manufacturer (none) -> YAGEO
- R8: renamed from R21; MPN (none) -> RC0805FR-0710KL; Manufacturer (none) -> YAGEO
- R9: renamed from R22; MPN (none) -> RC0805FR-0710KL; Manufacturer (none) -> YAGEO
Connections:
- net VBAT_OUT renamed VBAT_IN
