File: PowerSupply.kicad_sch (KiCad schematic)
At the start: 4 parts, among them U2 TPS62177DQC

Commit message: Inductance was replaced
Parts:
- C18: value TAJC686M010RNJ -> CA45-C010K107T
- L2: value 10uH -> KSE-CD5D18NP-220NC; footprint Inductor_SMD:L_6.3x6.3_H3 -> Inductor_SMD:L_Cenker_CKCS6028
Changed lines of the file:
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@@
 			)
 		)
-		(property "Value" "10uH"
+		(property "Value" "KSE-CD5D18NP-220NC"
 			(at 140.97 71.12 90)
 			(effects
@@
 			)
 		)
-		(property "Footprint" "Inductor_SMD:L_6.3x6.3_H3"
+		(property "Footprint" "Inductor_SMD:L_Cenker_CKCS6028"
 			(at 140.97 73.66 0)
 			(effects
@@
 			)
 		)
-		(property "Value" "TAJC686M010RNJ"
+		(property "Value" "CA45-C010K107T"
 			(at 161.29 80.3909 0)
 			(effects
