File: MCU.kicad_sch (KiCad schematic)
At the start: 38 parts, among them J10 UART1, J9 SWD, SW1 SM5-180UP-1, U5 STM32L072CBT6, Y1 4 MHz, Y2 32768 kHz

Commit message: Replace SIM800DC with A7682E
Connections:
- net UART2_DTR renamed RF_RESET
- net UART2_RI: no longer names the net of U5.39 (PB3)
- no-connect marks 9 -> 10
